File: Finalized-Boards/KLM_aux_SRAM/SRAM_exp.kicad_pcb (KiCad board)
At the start: 4 copper layers, 91 x 25.1 mm, 26 parts, among them J1 conn_80pin, J2 Conn_01x04, J3 Pmod_conn, U1 IS61WV204816BLL-10TLI, U2 LT1963AES8-3.3PBF

Commit message: Apply Matt's review changes to RTM, fanout and SRAM boards
SRAM: serial -> IDL_26_007 RevC - 09/2026 - CK/RS; vias untented (board-level);
GND zone 0.4 clearance / 0.1524 min width; In2 +3.3V stripe pulled back from
both board edges (tips 103.25 / 126.05) with 45-degree miters; +3.3V via moved
to (165.54, 125.92) and re-routed on F.Cu/B.Cu to clear GND (was 2 DRC errors);
C1/C2 0402 -> 0603 X7R in schematic and PCB; orphan teardrop + 2 zero-length
tracks removed.
Fanout: Matt's reworked layout (12 AWG input centred, both-side labels, 3 mm
shorter test points, D1/R1 as real reference designators, silk moved clear).
RTM: four 1812 1 A PPTCs, one per output; +5V pour full-board on F.Cu/In2,
GND on B.Cu/In1; 3.4 mm fused traces; zones extended past Edge.Cuts.
Removed stale pre-review gerbers/drills/layer PDFs (duplicates of Chris-Originals).
Parts:
- C1, C2: footprint Capacitor_SMD:C_0402_1005Metric -> Capacitor_SMD:C_0603_1608Metric
- moved C2 0.15 mm to (165.9, 104.3)
Routing:
- net +3.3V: track 30.1 -> 28.8 mm
Other:
- board text added: "IDL_26_007 RevC - 09/2026 - CK/RS"
- board text removed: "IDL_25_007 RevC - 03/2026 - CK"
