File: Finalized-Boards/KLM_aux_SRAM/SRAM_exp.kicad_pcb (KiCad board)
At the start: 4 copper layers, 91 x 25.1 mm, 26 parts, among them J1 conn_80pin, J2 Conn_01x04, J3 Pmod_conn, U1 IS61WV204816BLL-10TLI, U2 LT1963AES8-3.3PBF

Commit message: Matt's 9/17 review: RTM paired 5V/GND terminals, SRAM R1/R2 to 0603, fanout per-destination polyswitches; archive 9/16 boards
Parts:
- R1, R2: footprint Resistor_SMD:R_0402_1005Metric_Pad0.72x0.64mm_HandSolder -> Resistor_SMD:R_0603_1608Metric_Pad0.98x0.95mm_HandSolder
Routing:
- net /spare1: track 14.8 -> 14.2 mm
