File: Finalized-Boards/KLM_aux_SRAM/SRAM_exp.kicad_sch (KiCad schematic)
At the start: 23 parts, among them J1 conn_80pin, J2 Conn_01x04, J3 Pmod_conn, U1 IS61WV204816BLL-10TLI, U2 LT1963AES8-3.3PBF

Commit message: Apply Matt's review changes to RTM, fanout and SRAM boards
SRAM: serial -> IDL_26_007 RevC - 09/2026 - CK/RS; vias untented (board-level);
GND zone 0.4 clearance / 0.1524 min width; In2 +3.3V stripe pulled back from
both board edges (tips 103.25 / 126.05) with 45-degree miters; +3.3V via moved
to (165.54, 125.92) and re-routed on F.Cu/B.Cu to clear GND (was 2 DRC errors);
C1/C2 0402 -> 0603 X7R in schematic and PCB; orphan teardrop + 2 zero-length
tracks removed.
Fanout: Matt's reworked layout (12 AWG input centred, both-side labels, 3 mm
shorter test points, D1/R1 as real reference designators, silk moved clear).
RTM: four 1812 1 A PPTCs, one per output; +5V pour full-board on F.Cu/In2,
GND on B.Cu/In1; 3.4 mm fused traces; zones extended past Edge.Cuts.
Removed stale pre-review gerbers/drills/layer PDFs (duplicates of Chris-Originals).
Parts:
- C1, C2: footprint Capacitor_SMD:C_0402_1005Metric -> Capacitor_SMD:C_0603_1608Metric
Changed lines of the file:
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@@
 			)
 		)
-		(property "Footprint" "Capacitor_SMD:C_0402_1005Metric"
+		(property "Footprint" "Capacitor_SMD:C_0603_1608Metric"
 			(at 256.54 104.14 0)
 			(effects
@@
 			)
 		)
-		(property "Footprint" "Capacitor_SMD:C_0402_1005Metric"
+		(property "Footprint" "Capacitor_SMD:C_0603_1608Metric"
 			(at 182.88 101.6 0)
 			(effects

Commit message: Matt's 9/17 review: RTM paired 5V/GND terminals, SRAM R1/R2 to 0603, fanout per-destination polyswitches; archive 9/16 boards
Parts:
- R1, R2: footprint Resistor_SMD:R_0402_1005Metric_Pad0.72x0.64mm_HandSolder -> Resistor_SMD:R_0603_1608Metric_Pad0.98x0.95mm_HandSolder
Changed lines of the file:
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@@
 			)
 		)
-		(property "Footprint" "Resistor_SMD:R_0402_1005Metric_Pad0.72x0.64mm_HandSolder"
+		(property "Footprint" "Resistor_SMD:R_0603_1608Metric_Pad0.98x0.95mm_HandSolder"
 			(at 194.564 34.544 90)
 			(effects
@@
 			)
 		)
-		(property "Footprint" "Resistor_SMD:R_0402_1005Metric_Pad0.72x0.64mm_HandSolder"
+		(property "Footprint" "Resistor_SMD:R_0603_1608Metric_Pad0.98x0.95mm_HandSolder"
 			(at 181.864 34.544 90)
 			(effects

Commit message: Matt's 9/22 review: fanout fuses rotated, thermal-relief zones, stitching vias; SRAM footprints synced with library, sch/pcb parity fixed; add lib tables, schematic PDFs, full-severity DRC/ERC reports
Parts:
- H2: value ~ -> (none)
- J1: footprint CONN_5177985-3_TYC -> 1_My_footprint_lib:CONN_5177985-3_TYC
- U1: footprint 48L_TSOP-1_12X20_ISI -> 1_My_footprint_lib:48L_TSOP-1_12X20_ISI
